File: Keyboard.kicad_sch (KiCad schematic)
At the start: 95 parts, among them J2 USB_C, J3 USB_C_Receptacle_USB2.0_14P, J4 Conn_01x04_Pin, SW1 SW_Push, SW2 SW_Push, U1 STM32F303RETx, U2 USBLC6-2SC6, U3 AMS1117-3.3

Commit message: ibom v0 fixes
Parts:
- J3: value USB_C_Receptacle_USB2.0_14P -> USB_C
Changed lines of the file:
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@@
 			)
 		)
-		(property "Value" "USB_C_Receptacle_USB2.0_14P"
+		(property "Value" "USB_C"
 			(at 201.93 189.23 0)
 			(effects
